Commit message: fix: velodyne sensor plugin

File: prius_description/urdf/prius/prius.sdf.xacro (robot description, xacro)
@@ -664,4 +664,25 @@
     <!-- velodyne on the top -->
     <link name="top_lidar">
+      <pose>0 0 1.7 0 0 -1.579</pose>
+      <inertial>
+        <mass value="1.0"/>
+        <origin xyz="0 0 0.07212"/>
+        <inertia ixx="${(1.0 * (3.0*0.04267*0.04267 + 0.14424*0.14424)) / 12.0}" ixy="0" ixz="0"
+          iyy="${(1.0 * (3.0*0.04267*0.04267 + 0.14424*0.14424)) / 12.0}" iyz="0"
+          izz="${0.5 * 1.0 * (0.04267*0.04267)}"/>
+      </inertial>
+      <visual name="visual">
+        <geometry>
+          <mesh>
+          <uri>file://$(find prius_description)/models/velodyne/meshes/HDL32E_base.dae</uri>
+          </mesh>
+        </geometry>
+      </visual>
+      <collision name="collision">
+        <origin rpy="0 0 0" xyz="0 0 0.07212"/>
+        <geometry>
+          <cylinder radius="0.04267" length="0.14424"/>
+        </geometry>
+      </collision>
       <sensor name="gpu_lidar" type="gpu_lidar">
         <pose relative_to="chassis">0 0 1.7 0 0 -1.579</pose>
@@ -703,5 +724,4 @@
       <parent>chassis</parent>
       <child>top_lidar</child>
-      <pose>0 0 1.7 0 0 -1.579</pose>
     </joint>
     <!-- Ackermann Drive -->

Commit message: wip: bridge joint state properly

File: prius_description/urdf/prius/prius.sdf.xacro (robot description, xacro)
@@ -666,21 +666,21 @@
       <pose>0 0 1.7 0 0 -1.579</pose>
       <inertial>
-        <mass value="1.0"/>
-        <origin xyz="0 0 0.07212"/>
+        <mass value="1.0" />
+        <origin xyz="0 0 0.07212" />
         <inertia ixx="${(1.0 * (3.0*0.04267*0.04267 + 0.14424*0.14424)) / 12.0}" ixy="0" ixz="0"
           iyy="${(1.0 * (3.0*0.04267*0.04267 + 0.14424*0.14424)) / 12.0}" iyz="0"
-          izz="${0.5 * 1.0 * (0.04267*0.04267)}"/>
+          izz="${0.5 * 1.0 * (0.04267*0.04267)}" />
       </inertial>
       <visual name="visual">
         <geometry>
           <mesh>
-          <uri>file://$(find prius_description)/models/velodyne/meshes/HDL32E_base.dae</uri>
+            <uri>file://$(find prius_description)/models/velodyne/meshes/HDL32E_base.dae</uri>
           </mesh>
         </geometry>
       </visual>
       <collision name="collision">
-        <origin rpy="0 0 0" xyz="0 0 0.07212"/>
-        <geometry>
-          <cylinder radius="0.04267" length="0.14424"/>
+        <origin rpy="0 0 0" xyz="0 0 0.07212" />
+        <geometry>
+          <cylinder radius="0.04267" length="0.14424" />
         </geometry>
       </collision>
@@ -769,4 +769,15 @@
       </xacro:unless>
     </plugin>
+    <!-- Joints plugin -->
+    <plugin filename="gz-sim-joint-state-publisher-system"
+      name="gz::sim::systems::JointStatePublisher">
+      <xacro:if value="${namespace == '/'}">
+        <topic>prius/joint_state</topic>
+      </xacro:if>
+      <xacro:unless value="${namespace == '/'}">
+        <topic>${namespace}/prius/joint_state</topic>
+      </xacro:unless>
+      <update_rate>30</update_rate>
+    </plugin>
   </model>
 </sdf>

Commit message: wip: two 3d lidars :D

File: prius_description/urdf/prius/prius.sdf.xacro (robot description, xacro)
@@ -6,5 +6,5 @@
   <model name="prius_hybrid">
     <link name="base_link">
-      <pose>0 0 0 0 0 -1.59</pose>
+      <pose>0 1.45 0 0 0 -1.5708</pose>
     </link>
     <link name="chassis">
@@ -662,7 +662,7 @@
       <child>imu_link</child>
     </joint>
-    <!-- velodyne on the top -->
-    <link name="top_lidar">
-      <pose>0 0 1.7 0 0 -1.579</pose>
+    <!-- velodyne at the front -->
+    <link name="front_lidar">
+      <pose>0 -1.5 1.2 0 0.523 -1.5708</pose>
       <inertial>
         <mass value="1.0" />
@@ -685,6 +685,69 @@
         </geometry>
       </collision>
+      <sensor name="gpu_lidar_front" type="gpu_lidar">
+        <pose relative_to="chassis">0 -1.5 1.2 0 0.523 -1.5708</pose>
+        <xacro:if value="${namespace == '/'}">
+          <gz_frame_id>front_lidar</gz_frame_id>
+          <topic>front_lidar</topic>
+        </xacro:if>
+        <xacro:unless value="${namespace == '/'}">
+          <gz_frame_id>${namespace}/front_lidar</gz_frame_id>
+          <topic>${namespace}/front_lidar</topic>
+        </xacro:unless>
+        <update_rate>10</update_rate>
+        <ray>
+          <scan>
+            <horizontal>
+              <samples>640</samples>
+              <resolution>1</resolution>
+              <min_angle>-3.1</min_angle>
+              <max_angle>3.1</max_angle>
+            </horizontal>
+            <vertical>
+              <samples>32</samples>
+              <resolution>1</resolution>
+              <min_angle>-0.523</min_angle>
+              <max_angle>0.1745</max_angle>
+            </vertical>
+          </scan>
+          <range>
+            <min>0.08</min>
+            <max>130.0</max>
+            <resolution>0.01</resolution>
+          </range>
+        </ray>
+        <always_on>1</always_on>
+        <visualize>true</visualize>
+      </sensor>
+    </link>
+    <joint name="front_lidar_joint" type="fixed">
+      <parent>chassis</parent>
+      <child>front_lidar</child>
+    </joint>
+    <!-- velodyne on the top -->
+    <link name="top_lidar">
+      <pose>0 0 1.7 0 0 -1.5708</pose>
+      <inertial>
+        <mass value="1.0" />
+        <origin xyz="0 0 0.07212" />
+        <inertia ixx="${(1.0 * (3.0*0.04267*0.04267 + 0.14424*0.14424)) / 12.0}" ixy="0" ixz="0"
+          iyy="${(1.0 * (3.0*0.04267*0.04267 + 0.14424*0.14424)) / 12.0}" iyz="0"
+          izz="${0.5 * 1.0 * (0.04267*0.04267)}" />
+      </inertial>
+      <visual name="visual">
+        <geometry>
+          <mesh>
+            <uri>file://$(find prius_description)/models/velodyne/meshes/HDL32E_base.dae</uri>
+          </mesh>
+        </geometry>
+      </visual>
+      <collision name="collision">
+        <origin rpy="0 0 0" xyz="0 0 0.07212" />
+        <geometry>
+          <cylinder radius="0.04267" length="0.14424" />
+        </geometry>
+      </collision>
       <sensor name="gpu_lidar" type="gpu_lidar">
-        <pose relative_to="chassis">0 0 1.7 0 0 -1.579</pose>
+        <pose relative_to="chassis">0 0 1.7 0 0 -1.5708</pose>
         <xacro:if value="${namespace == '/'}">
           <gz_frame_id>top_lidar</gz_frame_id>
@@ -780,4 +843,11 @@
       <update_rate>30</update_rate>
     </plugin>
+    <!-- <plugin filename="libignition-gazebo-pose-publisher-system.so"  -->
+    <!--         name="gz::sim::systems::PosePublisher"> -->
+    <!--   <publish_link_pose>true</publish_link_pose> -->
+    <!--   <publish_collision_pose>false</publish_collision_pose> -->
+    <!--   <publish_visual_pose>false</publish_visual_pose> -->
+    <!--   <update_frequency>50</update_frequency> -->
+    <!-- </plugin> -->
   </model>
 </sdf>
